File: PCB/MMTK.kicad_pcb (KiCad board)
At the start: 4 copper layers, 135.5 x 60 mm, 100 parts, among them J2 Stepper, J3 LoadCell, J4 Barrel_Jack_Switch, J5 LCD, J7 ESTOP_SOFT, Q1 MMBT4403LT1G, Q2 Q_PMOS_GSD, Q3 2N7002, Q4 2N7002, Q5 2N7002, U1 HX711, U2 TMC2209, U3 TPS562200

Commit message: update and upgrade to kicad9
Other:
- net class Default removed
